File: pcb/infrared_row.sch (KiCad schematic (older format))
At the start: 17 parts, among them U2 QRE1113GR, U3 QRE1113GR, U4 QRE1113GR, U5 QRE1113GR, U6 QRE1113GR, U7 QRE1113GR, U8 QRE1113GR, U9 CD4051B

Commit message: Fix and Anotate design
Parts:
- gave numbers to parts that had none: 1
- renumbered C12 to C19

Commit message: MCU connections, OLED and Sonar
Parts:
- R53: footprint (none) -> Resistor_SMD:R_0805_2012Metric
