File: electrical/plugin_ir/infrared_row.sch (KiCad schematic (older format))
At the start: 17 parts, among them U2 QRE1113GR, U3 QRE1113GR, U4 QRE1113GR, U5 QRE1113GR, U6 QRE1113GR, U7 QRE1113GR, U8 QRE1113GR, U9 CD4051B

Commit message: Merge from master
Parts:
- renumbered C19 to C?, R6 to R?, R7 to R?, R8 to R?, R9 to R?, R10 to R?, R11 to R?, R12 to R?, R53 to R?, U9 to U?, U7 to U?, U6 to U?, U5 to U?, U4 to U?, U3 to U?, U2 to U?, U8 to U?
