File: electrical/core/power_supplies.sch (KiCad schematic (older format))
At the start: 30 parts, among them Q6 AO3400, U62 LM1117-ADJ, U63 TPS563200, U64 TPS62120

Commit message: Buck 3V3
Parts:
- added C38, C41: 0.1u, Capacitor_SMD:C_0603_1608Metric, symbol Device:C
- added C39, C40: 10u, Capacitor_SMD:C_0603_1608Metric, symbol Device:C
- added C42: 22p, Capacitor_SMD:C_0603_1608Metric, symbol Device:C
- added C43, C44: 22u, Capacitor_SMD:C_0603_1608Metric, symbol Device:C
- added L1: 3.3u, symbol Device:L
- added R94: 33k, Resistor_SMD:R_0603_1608Metric, symbol Device:R
- added R95: 10k, Resistor_SMD:R_0603_1608Metric, symbol Device:R
- added U63: TPS561201, Package_TO_SOT_SMD:SOT-23-8, symbol rasbot:TPS561201
- C45: renamed from C38; footprint (none) -> Capacitor_SMD:C_0603_1608Metric
- C51: renamed from C44; footprint (none) -> Capacitor_SMD:C_0603_1608Metric
- C52: renamed from C45; footprint (none) -> Capacitor_SMD:C_0603_1608Metric
- R91, R92, R93: footprint Capacitor_SMD:C_0603_1608Metric -> Resistor_SMD:R_0603_1608Metric
- R97: renamed from R95; footprint (none) -> Resistor_SMD:R_0603_1608Metric
- R99: renamed from R97; footprint (none) -> Resistor_SMD:R_0603_1608Metric
- renumbered C39 to C46, C40 to C47, C41 to C48, C42 to C49, C43 to C50, L1 to L2, L2 to L3, R98 to R100, R94 to R96, R96 to R98, U63 to U64, U64 to U65
Connections:
- net +BATT: now also C39.1, C40.1, C41.1, U63.3 (VIN), U63.5 (EN)
- net GND: now also C39.2, C40.2, C41.2, C43.2, C44.2, R95.2, U63.1 (GND)
- new net: C38.2, L1.1, U63.2 (SW)
- new net: C42.2, R94.1, R95.1, U63.4 (FB)
- new net: C38.1, U63.6 (VBST)
- new net: C42.1, C43.1, C44.1, L1.2, R94.2
Other:
- note added: "3V3 Buck"
