File: electrical/core/core.kicad_pcb (KiCad board)
At the start: 4 copper layers, 279 parts, among them J1 Conn_01x04, J10 ST-Link V2 Clones, J11 Segger J-Link SWD/JTAG, J12 ARM JTAG/SWD 10, J13 Expansion_Header_1, J14 Expansion_Header_2, J15 Expansion_Header_3, J16 Raspberry_Pi_2_3 IN, J17 Raspberry_Pi_2_3 OUT, J18 Conn_01x04_Male, J19 Conn_01x05_Male, J2 Conn_01x04_Male, J20 IR_Array_Power_Pass-through, J21 IR_Array_Slave_Link, J3 Conn_01x04_Male, J4 Conn_01x04_Male, J5 Conn_01x04_Male, J6 Conn_01x04_Male, J7 Conn_01x04_Male, J8 Conn_01x04_Male, J9 Conn_01x04_Male, M1 Motor_DC, M2 Motor_DC, M3 Motor_DC, M4 Motor_DC, Q1 AO3400, Q10 AO3400, Q11 AO3400, Q12 AO3400, Q13 AO3400, Q14 AO3400, Q15 AO3400, Q2 AO3400, Q3 AO3400, Q4 AO3400, Q5 AO3400, Q6 AO3400, Q7 AO3400, Q8 AO3400, Q9 AO3400, SW1 RESET, U1 DRV8874-Q1, U10 STM32F469BITx, U11 24LC256, U12 CAT4103V, U13 CAT4103V, U14 CAT4103V, U15 CAT4103V, U16 DRV8874-Q1, U17 MCP41HV51, U18 DRV8874-Q1, U19 MCP41HV51, U2 MCP41HV51, U3 DRV8874-Q1, U4 MCP41HV51, U5 TPS62120, U6 TPS561201, U7 TPS566235RJNx, U8 BQ76925, U9 BMX055, Y1 32.768KHz, Y2 25MHz

Commit message: Updated doc and reorganization of components in main board layout
Parts:
- moved C13 995.9 mm to (-791.3, -254.7)
- moved C16 995.9 mm to (-804.0, -254.9)
- moved C18 995.9 mm to (-772.0, -255.4)
- moved C27 995.9 mm to (-782.5, -276.4)
- moved C29 995.9 mm to (-750.8, -244.5)
- moved L3 995.9 mm to (-770.0, -241.2)
- moved R13 995.9 mm to (-764.7, -265.5)
- moved R15 995.9 mm to (-789.8, -201.1)
- moved TP5 995.9 mm to (-795.2, -264.5)
- moved TP6 995.9 mm to (-778.3, -264.5)
- moved U7 995.9 mm to (-788.8, -236.4)
- moved C20 995.9 mm to (-814.5, -242.2)
- moved C25 995.9 mm to (-757.2, -262.9)
- moved C30 995.9 mm to (-793.7, -273.2)
- moved C31 995.9 mm to (-757.0, -278.1)
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Other:
- board text added: "5V Buck Sonar"
- board text added: "Expansion Header"
- board text added: "MCU"
- board text added: "Power LED"
- board text added: "Reset"
- board text removed: "5V Sonar"

Commit message: BMS layout try
Parts:
- removed TP7, TP8: TestPoint, TestPoint:TestPoint_Pad_D1.0mm
- added TP28: TP_I2C2_SDA, TestPoint:TestPoint_Pad_D1.0mm, F.Cu at (130.3, -417.3)
- added TP29: TP_I2C2_SCL, TestPoint:TestPoint_Pad_D1.0mm, F.Cu at (133.4, -417.3)
- added TP_Cell2: TestPoint, TestPoint:TestPoint_Pad_D1.0mm, F.Cu at (370.5, -571.3)
- added TP_Cell3: TestPoint, TestPoint:TestPoint_Pad_D1.0mm, F.Cu at (363.4, -571.2)
- C26: moved to B.Cu
- TP23: value TestPoint -> TP_I2C1_SCL
- TP25: value TestPoint -> TP_I2C1_SDA
- moved R24 1343.8 mm to (355.8, -562.7), turned to 270 degrees
- moved C37 1326.3 mm to (345.3, -587.2), turned to 90 degrees
- moved R20 1322.8 mm to (365.2, -578.1)
- moved TP_BATT+1 1322.7 mm to (349.9, -598.1)
- moved C35 1322.3 mm to (345.3, -590.4), turned to 90 degrees
- moved R23 1321.7 mm to (332.3, -562.6), turned to 270 degrees
- moved BT1 1321.5 mm to (356.9, -598.2), turned to 90 degrees
- moved TP_Cell0 1321.3 mm to (370.5, -566.6)
- moved TP_Cell1 1319.7 mm to (363.5, -566.6)
- moved R25 1319.4 mm to (333.1, -571.6)
- moved R19 1319.3 mm to (365.2, -580.9)
- moved C42 1319.0 mm to (332.3, -567.1), turned to 90 degrees
- moved R21 1317.8 mm to (340.5, -573.1), turned to 270 degrees
- moved C43 1315.9 mm to (343.5, -565.9), turned to 270 degrees
- moved R18 1315.0 mm to (365.2, -583.8)
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- renumbered TP12 to TP_BATT+1, TP10 to TP_Cell0, TP9 to TP_Cell1, TP11 to TP_TH1
Connections:
- TP23 pad 1: /I2C1_SDA -> /I2C1_SCL
- TP25 pad 1: /I2C1_SCL -> /I2C1_SDA
Routing:
- net -BATT: track 0.00 -> 70.1 mm, vias 0 -> 3
- net Net-(C33-Pad2): track 0.00 -> 55.3 mm, vias 0 -> 2
- net Net-(C32-Pad1): track 0.00 -> 51.8 mm, vias 0 -> 2
- net Net-(C32-Pad2): track 0.00 -> 48.6 mm, vias 0 -> 2
- net Net-(C36-Pad1): track 0.00 -> 45.1 mm, vias 0 -> 2
- net /Battery_Current: track 0.00 -> 37.5 mm, vias 0 -> 1
- net /Power/Cell3: track 0.00 -> 35.6 mm
- net /Battery_Overcurrent: track 0.00 -> 32.0 mm, vias 0 -> 1
- net Net-(C42-Pad1): track 0.00 -> 30.9 mm, vias 0 -> 2
- net /Vref_opt: track 0.00 -> 30.7 mm, vias 0 -> 1
- net /Battery_Cell_Voltage: track 0.00 -> 29.5 mm, vias 0 -> 1
- net Net-(R22-Pad2): track 0.00 -> 26.7 mm
- net Net-(C42-Pad2): track 0.00 -> 24.1 mm, vias 0 -> 2
- net GND: track 0.00 -> 23.5 mm
- net /I2C1_SDA: track 0.00 -> 19.5 mm, vias 0 -> 1
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- added copper zone on PWR, net +BATT
- added copper zone on GND, net -BATT

Commit message: Motor 1 try layout
Parts:
- C2, JP2, JP3, R2, R3: moved to B.Cu
- moved JP2 515.0 mm to (503.3, -702.2), turned to 270 degrees
- moved M1 512.1 mm to (497.7, -676.8)
- moved C3 508.1 mm to (507.0, -687.4), turned to 270 degrees
- moved Q1 507.3 mm to (491.8, -691.1), turned to 90 degrees
- moved C10 507.2 mm to (529.0, -606.9)
- moved JP16 507.2 mm to (601.7, -598.5)
- moved JP18 507.2 mm to (601.7, -594.9)
- moved C87 507.2 mm to (602.3, -601.9)
- moved C90 507.2 mm to (609.9, -593.8)
- moved C91 507.2 mm to (609.9, -598.8)
- moved JP17 507.2 mm to (607.3, -601.8)
- moved JP4 507.2 mm to (509.6, -610.8)
- moved JP5 507.2 mm to (510.0, -603.6)
- moved M2 507.2 mm to (551.6, -596.9)
- moved Q15 507.2 mm to (610.1, -608.0)
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Routing:
- net +BATT: track 12.8 -> 130.4 mm
- net GND: track 23.5 -> 62.1 mm, vias 0 -> 4
- net +3V3: track 0.00 -> 30.2 mm, vias 0 -> 3
- net /D1_nFAULT: track 0.00 -> 24.3 mm, vias 0 -> 1
- net /D1_DigiPot_CS: track 0.00 -> 24.2 mm, vias 0 -> 1
- net /SPI2_SCK: track 0.00 -> 21.6 mm, vias 0 -> 1
- net Net-(M1-Pad2): track 0.00 -> 20.7 mm, vias 0 -> 2
- net /SPI2_MOSI: track 0.00 -> 19.1 mm, vias 0 -> 1
- net /D1_PMODE: track 0.00 -> 19.1 mm
- net /SPI2_MISO: track 0.00 -> 18.8 mm, vias 0 -> 1
- net /D1_DigiPot_WLAT: track 0.00 -> 18.6 mm, vias 0 -> 1
- net /D1_DigiPot_SHDN: track 0.00 -> 18.4 mm, vias 0 -> 1
- net Net-(M1-Pad1): track 0.00 -> 17.7 mm, vias 0 -> 2
- net /D1_SENSE: track 0.00 -> 17.0 mm, vias 0 -> 1
- net /D1_IMODE: track 0.00 -> 16.9 mm, vias 0 -> 1
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- added copper zone on PWR, net +3V3
- added copper zone on GND, net GND
